File: Rev. 2/Eagle/C64-Wifi_UserP.brd (EAGLE design)
At the start: 53.3 x 59 mm, 51 parts, among them IC1 74HC14D, J1 C64-USERPORT, J2 n/a, M1 NODEMCUV3COMBI, Q1 BSS138, Q2 BSS138, Q3 BSS138, Q4 BSS138, Q5 BSS138, Q6 BC846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

Commit message: Silk Screen Update
Parts:
- added U$45: OPEN_SOURCE_HW, Logo:OPENHW
Other:
- board text added: "100n"
- board text added: "10k"
- board text added: "2x 41 48"
- board text added: "3x 330R"
- board text added: "3x330R"
- board text added: "5x BSS138"
- board text added: "5x10k"
- board text added: "74HC14D"
- board text added: "BAT54"
- board text added: "BC846"
- board text added: "http://github.com/ svenpetersen1965"
Changed lines of the file:
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@@
 <layer number="25" name="tNames" color="7" fill="1" visible="yes" active="yes"/>
 <layer number="26" name="bNames" color="7" fill="1" visible="no" active="yes"/>
-<layer number="27" name="tValues" color="7" fill="1" visible="no" active="yes"/>
+<layer number="27" name="tValues" color="62" fill="1" visible="no" active="yes"/>
 <layer number="28" name="bValues" color="7" fill="1" visible="no" active="yes"/>
 <layer number="29" name="tStop" color="7" fill="3" visible="no" active="yes"/>
@@
 <layer number="250" name="Descript" color="7" fill="1" visible="no" active="no"/>
 <layer number="251" name="SMDround" color="7" fill="1" visible="no" active="no"/>
+<layer number="252" name="BR-BS" color="7" fill="1" visible="no" active="yes"/>
+<layer number="253" name="BR-LS" color="7" fill="1" visible="no" active="yes"/>
 <layer number="254" name="OrgLBR" color="7" fill="1" visible="no" active="no"/>
 <layer number="255" name="Accent" color="7" fill="1" visible="no" active="yes"/>
@@
 <dimension x1="50.00625" y1="53.34" x2="54.2925" y2="46.51375" x3="55.245" y3="46.51375" textsize="1.016" textratio="12" layer="47" dtype="leader"/>
 <text x="55.88" y="46.0375" size="1.016" layer="47" ratio="12">3.3</text>
+<text x="50.64125" y="29.05125" size="1.27" layer="22" rot="MR0">http://github.com/
+svenpetersen1965</text>
+<text x="4.1275" y="34.13125" size="1.016" layer="21">100n</text>
+<text x="7.9375" y="30.63875" size="1.27" layer="21">74HC14D</text>
+<text x="6.0325" y="38.25875" size="1.016" layer="21">3x 330R</text>
+<text x="18.89125" y="35.8775" size="1.016" layer="21">100n</text>
+<text x="22.86" y="35.8775" size="1.016" layer="21">10k</text>
+<text x="25.7175" y="25.4" size="1.016" layer="21">10k</text>
+<text x="14.76375" y="24.92375" size="1.016" layer="21">100n</text>
+<text x="24.13" y="28.41625" size="1.016" layer="21">2x
+41
+48</text>
+<text x="26.3525" y="35.71875" size="1.27" layer="21">BC846</text>
+<text x="26.3525" y="29.68625" size="1.27" layer="21">BC846</text>
+<text x="8.5725" y="12.3825" size="1.016" layer="21">5x10k</text>
+<text x="8.5725" y="7.3025" size="1.016" layer="21">5x10k</text>
+<text x="8.5725" y="8.89" size="1.016" layer="21">5x
+BSS138</text>
+<text x="36.83" y="57.4675" size="1.27" layer="21">BC846</text>
+<text x="41.43375" y="51.27625" size="1.27" layer="21" rot="R90">10k</text>
+<text x="31.115" y="56.99125" size="1.016" layer="21">3x330R</text>
+<text x="35.2425" y="16.51" size="1.27" layer="21">BAT54</text>
 </plain>
 <attributes>
@@
 <element name="Q2" library="Transistoren" package="SOT23" value="BSS138" x="16.25625" y="10.795" smashed="yes" rot="R180">
 <attribute name="NAME" x="14.51" y="10.00125" size="1.27" layer="25" rot="R90"/>
-<attribute name="VALUE" x="13.0175" y="13.5575" size="1.27" layer="27" rot="R270"/>
+<attribute name="VALUE" x="18.415" y="14.1925" size="1.27" layer="27" rot="R270"/>
 </element>
 <element name="Q3" library="Transistoren" package="SOT23" value="BSS138" x="25.24125" y="10.795" smashed="yes" rot="R180">
@@
 <element name="D1" library="Dioden" package="SOD80C" value="LL4148" x="19.28875" y="31.47125" smashed="yes">
 <attribute name="NAME" x="21.68905" y="30.6775" size="1.27" layer="25" ratio="10"/>
-<attribute name="VALUE" x="20.41905" y="30.7537" size="1.016" layer="27" ratio="10"/>
+<attribute name="VALUE" x="20.10155" y="31.54745" size="0.8128" layer="27" ratio="10"/>
 </element>
 <element name="D2" library="Dioden" package="SOD80C" value="LL4148" x="19.28875" y="29.23375" smashed="yes">
 <attribute name="NAME" x="21.68905" y="28.59875" size="1.27" layer="25" ratio="10"/>
-<attribute name="VALUE" x="20.41905" y="28.67495" size="1.016" layer="27" ratio="10"/>
+<attribute name="VALUE" x="20.10155" y="28.35745" size="0.8128" layer="27" ratio="10"/>
 </element>
 <element name="C2" library="SMD" package="0805" value="100n" x="19.765" y="33.6" smashed="yes">
@@
 </element>
 <element name="Q6" library="Transistoren" package="SOT23" value="BC846" x="27.54375" y="34.205" smashed="yes">
-<attribute name="NAME" x="25.95625" y="35.7925" size="1.27" layer="25"/>
-<attribute name="VALUE" x="25.95625" y="35.7925" size="1.27" layer="27"/>
+<attribute name="NAME" x="29.29" y="33.57" size="1.27" layer="25"/>
+<attribute name="VALUE" x="26.4325" y="35.7925" size="1.27" layer="27"/>
 </element>
 <element name="Q7" library="Transistoren" package="SOT23" value="BC846" x="27.385" y="28.09375" smashed="yes">
-<attribute name="NAME" x="30.485" y="27.22625" size="1.27" layer="25" rot="R90"/>
-<attribute name="VALUE" x="25.7975" y="29.68125" size="1.27" layer="27"/>
+<attribute name="NAME" x="29.13125" y="27.6175" size="1.27" layer="25"/>
+<attribute name="VALUE" x="26.27375" y="29.68125" size="1.27" layer="27"/>
 </element>
 <element name="R18" library="SMD" package="0805" value="330R" x="32.6225" y="55.7725" smashed="yes" rot="R180">
@@
 <element name="D3" library="Dioden" package="SOT23" value="BAT54" x="33.416875" y="17.383125" smashed="yes" rot="R270">
 <attribute name="NAME" x="34.210625" y="18.018125" size="1.27" layer="25"/>
-<attribute name="VALUE" x="35.163125" y="17.383125" size="1.27" layer="27"/>
+<attribute name="VALUE" x="35.163125" y="16.589375" size="1.27" layer="27"/>
 </element>
 <element name="SW1" library="Namae_Electronics" package="JTP-1130" value="JTP-1130" x="49.3" y="12.8" smashed="yes" rot="R90">
@@
 <element name="DRL2" library="Mech_Bohr" package="BOHR3,3" value="" x="4" y="12.8" smashed="yes"/>
 <element name="U$44" library="Logo" package="SVEN_TAG" value="" x="35.71875" y="32.385" smashed="yes"/>
+<element name="U$45" library="Logo" package="OPENHW" value="OPEN_SOURCE_HW" x="50.64125" y="33.3375" smashed="yes" rot="MR0"/>
 </elements>
 <signals>
