File: Rev. 2/Eagle/C64-Wifi_UserP.sch (EAGLE design)
At the start: 46 parts, among them IC1 74HC14D, J1 C64-USERPORT, J2 n/a, M1 NODEMCUV3COMBI, Q1 BSS138, Q2 BSS138, Q3 BSS138, Q4 BSS138, Q5 BSS138, Q6 BC846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

Commit message: Silk Screen Update
Parts:
- added U$45: OPEN_SOURCE_HW, Logo:OPEN_SOURCE_HW
Other:
- note added: "http://github.com/svenpetersen1965"
- note added: "tact switch 6x6mm"
- note removed: "e.g. Kingbright KP-2012SURC Reichelr KBT KP-2012SURC"
- moved on the sheet: IC1P
Changed lines of the file:
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@@
 <layer number="250" name="Descript" color="7" fill="1" visible="no" active="no"/>
 <layer number="251" name="SMDround" color="7" fill="1" visible="no" active="no"/>
+<layer number="252" name="BR-BS" color="7" fill="1" visible="no" active="yes"/>
+<layer number="253" name="BR-LS" color="7" fill="1" visible="no" active="yes"/>
 <layer number="254" name="OrgLBR" color="7" fill="1" visible="no" active="no"/>
 <layer number="255" name="Accent" color="7" fill="1" visible="yes" active="yes"/>
@@
 <part name="DRL1" library="Mech_Bohr" deviceset="BOHR3,3" device=""/>
 <part name="DRL2" library="Mech_Bohr" deviceset="BOHR3,3" device=""/>
+<part name="U$45" library="Logo" deviceset="OPEN_SOURCE_HW" device=""/>
 </parts>
 <sheets>
@@
 <text x="347.98" y="22.86" size="2.54" layer="95">Sven Petersen</text>
 <text x="340.36" y="17.78" size="2.54" layer="95">2</text>
-<text x="274.32" y="132.08" size="1.6764" layer="96">e.g. Kingbright
-KP-2012SURC
-Reichelr KBT KP-2012SURC</text>
 <text x="99.06" y="142.24" size="1.6764" layer="96">on precision socket strips:
 2x MPE 115-1-015
@@
 (25.4mm and 31.3mm width)
 fit the footprint on the PCB. </text>
+<text x="279.4" y="7.62" size="2.54" layer="95">http://github.com/svenpetersen1965</text>
+<text x="323.85" y="156.21" size="1.778" layer="96">tact switch
+6x6mm</text>
 </plain>
 <instances>
@@
 <attribute name="NAME" x="48.895" y="48.895" size="1.778" layer="95"/>
 </instance>
+<instance part="U$45" gate="G$1" x="238.76" y="7.62" smashed="yes"/>
 </instances>
 <busses>
@@
 <pinref part="U$26" gate="1" pin="GND"/>
 <pinref part="IC1" gate="P" pin="GND"/>
-<wire x1="156.21" y1="40.64" x2="156.21" y2="43.18" width="0.1524" layer="91"/>
+<wire x1="156.21" y1="40.64" x2="156.21" y2="44.45" width="0.1524" layer="91"/>
 </segment>
 <segment>
@@
 <pinref part="IC1" gate="P" pin="VCC"/>
 <pinref part="U$24" gate="1" pin="+5V"/>
-<wire x1="156.21" y1="55.88" x2="156.21" y2="58.42" width="0.1524" layer="91"/>
-<wire x1="156.21" y1="55.88" x2="166.37" y2="55.88" width="0.1524" layer="91"/>
-<junction x="156.21" y="55.88"/>
+<wire x1="156.21" y1="57.15" x2="156.21" y2="58.42" width="0.1524" layer="91"/>
+<wire x1="156.21" y1="57.15" x2="166.37" y2="57.15" width="0.1524" layer="91"/>
+<junction x="156.21" y="57.15"/>
 <pinref part="C1" gate="G$1" pin="2"/>
-<wire x1="166.37" y1="55.88" x2="166.37" y2="50.8" width="0.1524" layer="91"/>
-</segment>
-<segment>
+<wire x1="166.37" y1="57.15" x2="166.37" y2="50.8" width="0.1524" layer="91"/>
+</segment>
+<segment>
